File: hw/brd/kom.sch (KiCad schematic (older format))
At the start: 90 parts, among them IC1 ATMEGA328-P, IC2 4067D, IC3 L293D, J1 ExtPwr, M1 XBEE, P1 Batt, P10 IR_Scanner, P11 GPIO_4PIN, P12 GPIO_4PIN, P13 GPIO_4PIN, P14 GPIO_4PIN, P15 GPIO_4PIN, P16 GPIO_4PIN, P17 GPIO_4PIN, P18 GPIO_4PIN, P2 Serial, P3 ICSP, P4 GPIO_4PIN, P5 GPIO_4PIN, P6 GPIO_4PIN, P7 GPIO_4PIN, P8 GPIO_4PIN, P9 GPIO_4PIN, Q1 PT480F, Q2 PT480F, Q3 PT480F, Q4 PT480F, SW1 SW_PUSH, SW2 PwrSelect, SW3 PWR_Control, SW4 TEST, U1 LM7833, U2 74LS125, U3 TC54, U4 PTH08000WAZT, U5 ULN2003A, X1 16MHz

Commit message: Changed some schematic symbols for the ones found in Monolito. Added bypass capacitors
Parts:
- removed I2C1, I2C2: CONN_4, symbol CONN_4
- removed J1: ExtPwr, symbol JACK_2P
- removed P3: ICSP, symbol CONN_3X2
- added BypC?: IR, symbol CPOL
- added BypC?: H, symbol CPOL
- added BypC?: Servo, symbol CPOL
- added BypC?: US, symbol CPOL
- added BypC?: Mux, symbol CPOL
- added H1: HEAD3X2, symbol HEAD3X2
- added J?1: EXT, symbol JACK
- added JP2, JP3: JP_4, symbol JP_4
Connections:
- wire segments 235 -> 248
Other:
- note added: "GPIOs"
- moved on the sheet: C2, C6, CP1, CP2, D1, D3, F1, P4, P5, P6, P7, P8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

Commit message: New BOM, including the URLs to Farnell components
Parts:
- D3: value LED -> UVLO
- H1: value HEAD3X2 -> ICSP
- SW1: value SW_PUSH -> SW_RESET
- gave numbers to parts that had none: 5
- renumbered JP3 to I2C, JP2 to I2C
Changed lines of the file:
@@
-EESchema Schematic File Version 2  date Thu 21 Jun 2012 11:50:03 AM CEST
+EESchema Schematic File Version 2  date Thu 21 Jun 2012 04:38:35 PM CEST
 LIBS:power
 LIBS:device
@@
 P 3950 2200
 F 0 "D3" H 3950 2300 50  0000 C CNN
-F 1 "LED" H 3950 2100 50  0000 C CNN
+F 1 "UVLO" H 3950 2100 50  0000 C CNN
 	1    3950 2200
 	1    0    0    -1
@@
 P 1800 5250
 F 0 "SW1" H 1950 5360 50  0000 C CNN
-F 1 "SW_PUSH" H 1800 5170 50  0000 C CNN
+F 1 "SW_RESET" H 1800 5170 50  0000 C CNN
 	1    1800 5250
 	0    -1   -1   0
@@
 P 1300 5950
 F 0 "H1" H 1650 6100 60  0000 C CNN
-F 1 "HEAD3X2" H 1800 5600 40  0000 C CNN
+F 1 "ICSP" H 1800 5600 40  0000 C CNN
 	1    1300 5950
 	1    0    0    -1
 $EndComp
 $Comp
-L JP_4 JP3
+L JP_4 I2C
 U 1 1 4FE2F5BD
 P 2750 9800
-F 0 "JP3" H 2910 10020 60  0000 C CNN
+F 0 "I2C" H 2910 10020 59  0000 C CNN
 F 1 "JP_4" H 2900 9740 60  0001 C CNN
 	1    2750 9800
@@
 $EndComp
 $Comp
-L JP_4 JP2
+L JP_4 I2C
 U 1 1 4FE2F5D4
 P 2250 9800
-F 0 "JP2" H 2410 10020 60  0000 C CNN
+F 0 "I2C" H 2410 10020 59  0000 C CNN
 F 1 "JP_4" H 2400 9740 60  0001 C CNN
 	1    2250 9800
@@
 GPIOs
 $Comp
-L OSHW-LOGO #G?
+L OSHW-LOGO #G1
 U 1 1 4FE2FC53
 P 11450 10800
-F 0 "#G?" H 11450 10497 60  0001 C CNN
+F 0 "#G1" H 11450 10497 60  0001 C CNN
 F 1 "OSHW-LOGO" H 11450 11103 60  0001 C CNN
 	1    11450 10800
@@
 $EndComp
 $Comp
-L CPOL BypC?
+L CPOL BypC1
 U 1 1 4FE2FF65
 P 7900 6600
-F 0 "BypC?" H 7950 6750 50  0000 L CNN
+F 0 "BypC1" H 7950 6750 50  0000 L CNN
 F 1 "IR" H 8000 6450 50  0000 L CNN
 	1    7900 6600
@@
 $EndComp
 $Comp
-L CPOL BypC?
+L CPOL BypC2
 U 1 1 4FE2FF90
 P 8350 6600
-F 0 "BypC?" H 8400 6750 50  0000 L CNN
+F 0 "BypC2" H 8400 6750 50  0000 L CNN
 F 1 "H" H 8450 6450 50  0000 L CNN
 	1    8350 6600
@@
 $EndComp
 $Comp
-L CPOL BypC?
+L CPOL BypC3
 U 1 1 4FE2FF96
 P 8800 6600
-F 0 "BypC?" H 8850 6750 50  0000 L CNN
+F 0 "BypC3" H 8850 6750 50  0000 L CNN
 F 1 "Servo" H 8900 6450 50  0000 L CNN
 	1    8800 6600
@@
 $EndComp
 $Comp
-L CPOL BypC?
+L CPOL BypC4
 U 1 1 4FE2FFB0
 P 9250 6600
-F 0 "BypC?" H 9300 6750 50  0000 L CNN
+F 0 "BypC4" H 9300 6750 50  0000 L CNN
 F 1 "US" H 9350 6450 50  0000 L CNN
 	1    9250 6600
@@
 $EndComp
 $Comp
-L CPOL BypC?
+L CPOL BypC5
 U 1 1 4FE2FFB6
 P 9700 6600
-F 0 "BypC?" H 9750 6750 50  0000 L CNN
+F 0 "BypC5" H 9750 6750 50  0000 L CNN
 F 1 "Mux" H 9800 6450 50  0000 L CNN
 	1    9700 6600
@@
 Connection ~ 8350 6700
 $Comp
-L +5V #PWR?
+L +5V #PWR065
 U 1 1 4FE31ED6
 P 8800 6050
-F 0 "#PWR?" H 8800 6140 20  0001 C CNN
+F 0 "#PWR065" H 8800 6140 20  0001 C CNN
 F 1 "+5V" H 8800 6140 30  0000 C CNN
 	1    8800 6050
@@
 $EndComp
 $Comp
-L GND #PWR?
+L GND #PWR066
 U 1 1 4FE31EE5
 P 8800 6800
-F 0 "#PWR?" H 8800 6800 30  0001 C CNN
+F 0 "#PWR066" H 8800 6800 30  0001 C CNN
 F 1 "GND" H 8800 6730 30  0001 C CNN
 	1    8800 6800

Commit message: Before merging
Parts:
- renumbered I2C to I2C1, I2C to I2C2

Commit message: - Using a single barrel connector for power input. - Added Inverse Polarity Protection (IPP) with fuse + crowbar diode. TEST IT!!! - Added On LED
Parts:
- removed P1: Batt, symbol CONN_2
- added D11: LED, symbol LED
- added R23: 330, symbol R
- D1: value DIODE -> InvPolarity
- SW2: value PwrSelect -> PwrOn
Connections:
- net labels removed: ExtIn
- wire segments 248 -> 245
- no-connect marks 15 -> 16
Other:
- moved on the sheet: J?1

Commit message: Small fixes
Parts:
- D11: value LED -> ON
Other:
- note added: "Test the IPP!"
Changed lines of the file:
@@
-EESchema Schematic File Version 2  date Fri 22 Jun 2012 08:11:17 PM CEST
+EESchema Schematic File Version 2  date Fri 22 Jun 2012 08:13:31 PM CEST
 LIBS:power
 LIBS:device
@@
 P 6750 2300
 F 0 "D11" H 6750 2400 50  0000 C CNN
-F 1 "LED" H 6750 2200 50  0000 C CNN
+F 1 "ON" H 6750 2200 50  0000 C CNN
 	1    6750 2300
 	0    1    1    0
@@
 	1    0    0    -1
 $EndComp
+Text Notes 2450 2100 0    58   Italic 12
+Test the IPP!
 $EndSCHEMATC

Commit message: Minor changes
Other:
- note added: "Not all caps go to +5V!"
Changed lines of the file:
@@
-EESchema Schematic File Version 2  date Fri 22 Jun 2012 08:13:31 PM CEST
+EESchema Schematic File Version 2  date Fri 22 Jun 2012 08:22:02 PM CEST
 LIBS:power
 LIBS:device
@@
 Text Notes 2450 2100 0    58   Italic 12
 Test the IPP!
+Text Notes 9750 6100 0    58   Italic 12
+Not all caps go to +5V!
 $EndSCHEMATC

Commit message: - Changed to JST-XH connector for LiPo - Changed and added bypass capacitors - LC filter on AVCC
Parts:
- removed BypC1: IR, symbol CPOL
- removed C2, C6: 100uF(min), symbol C
- added 10uH1: INDUCTOR, symbol INDUCTOR
- added AVCC_Cap1, AVR_Cap1: 100n, symbol C
- added BypCCap1: MotorL, symbol C
- added BypCCap2: MotorR, symbol C
- added InCap1: 100uF, symbol CPOL
- added K1: CONN_3, symbol CONN_3
- added RadioCCap1: 8.2pF, symbol C
- added RadioECap1: 1uF, symbol CPOL
- H_Cap1: renamed from BypC2; value H -> 100uF
- IR_Cap1: renamed from BypC3; value Servo -> 10uF
- Mux_Cap1: renamed from BypC5; value Mux -> 100nF
- US_Cap1: renamed from BypC4; value US -> 10uF
- renumbered C3 to C2, C4 to C3, C5 to C4, D9 to D10, D10 to D11, D11 to D4, D4 to D5, D5 to D6, D6 to D7, D7 to D8, D8 to D9, I2C1 to I1, I2C2 to I2, J?1 to J1, P2 to P1, P12 to P10, P13 to P11, P14 to P12, P15 to P13, P16 to P14, P17 to P15, P18 to P16, P4 to P2, P5 to P3, P6 to P4, P7 to P5, P8 to P6, P9 to P7, P10 to P8, P11 to P9, R9 to R10, R10 to R11, R11 to R12, R12 to R13, R13 to R14, R14 to R16, R16 to R17, R17 to R18, R18 to R19, R19 to R20, R20 to R21, R21 to R22, R22 to R23, R5 to R4, R6 to R5, R4 to R6, R23 to R9
Connections:
- net labels added: AVCC
- wire segments 245 -> 350
Other:
- note added: "Decoupling Capacitors"
- note removed: "Not all caps go to +5V!"
- moved on the sheet: BT1, CP1, CP2, CP3, CP4, D5, D6, D7, D8, H_Cap1, IC3, IR_Cap1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

Commit message: Before footprint asociation
Parts:
- F1: value FUSE -> 1.1A Fuse
- InvPolDiode1: renamed from D1; value InvPolarity -> 200mA min
- renumbered D2 to D1, D11 to D10, D3 to D2, D4 to D3, D5 to D4, D6 to D5, D7 to D6, D8 to D7, D9 to D8, D10 to D9, 10uH1 to U1, U1 to U2, U2 to U3, U3 to U4, U4 to U5, U5 to U6
Other:
- note removed: "Test the IPP!"
Changed lines of the file:
@@
-EESchema Schematic File Version 2  date Mon 25 Jun 2012 02:42:49 PM CEST
+EESchema Schematic File Version 2  date Mon 25 Jun 2012 06:43:30 PM CEST
 LIBS:power
 LIBS:device
@@
 $EndComp
 $Comp
-L PTH08000WAZT U4
+L PTH08000WAZT U5
 U 1 1 4FCE13E4
 P 5800 1900
-F 0 "U4" H 5800 1500 60  0000 C CNN
+F 0 "U5" H 5800 1500 60  0000 C CNN
 F 1 "PTH08000WAZT" H 5800 2150 60  0000 C CNN
 	1    5800 1900
@@
 $EndComp
 $Comp
-L LED D3
+L LED D2
 U 1 1 4FCE13F0
 P 3950 2200
-F 0 "D3" H 3950 2300 50  0000 C CNN
+F 0 "D2" H 3950 2300 50  0000 C CNN
 F 1 "UVLO" H 3950 2100 50  0000 C CNN
 	1    3950 2200
@@
 $EndComp
 $Comp
-L TC54 U3
+L TC54 U4
 U 1 1 4FCE13F6
 P 3950 2550
-F 0 "U3" H 4100 2300 60  0000 C CNN
+F 0 "U4" H 4100 2300 60  0000 C CNN
 F 1 "TC54" H 3950 2650 60  0000 C CNN
 	1    3950 2550
@@
 P 3100 1800
 F 0 "F1" H 3200 1850 40  0000 C CNN
-F 1 "FUSE" H 3000 1750 40  0000 C CNN
+F 1 "1.1A Fuse" H 3100 1700 40  0000 C CNN
 	1    3100 1800
 	0    -1   -1   0
@@
 $EndComp
 $Comp
-L 74LS125 U2
+L 74LS125 U3
 U 1 1 4FD32B86
 P 3600 9050
-F 0 "U2" H 3600 9150 50  0000 L BNN
+F 0 "U3" H 3600 9150 50  0000 L BNN
 F 1 "74LS125" H 3650 8900 40  0000 L TNN
 	1    3600 9050
@@
 $EndComp
 $Comp
-L LM7805 U1
+L LM7805 U2
 U 1 1 4FD32BAA
 P 3550 8200
-F 0 "U1" H 3700 8004 60  0000 C CNN
+F 0 "U2" H 3700 8004 60  0000 C CNN
 F 1 "LM7833" H 3550 8400 60  0000 C CNN
 	1    3550 8200
@@
 AT_DIN
 $Comp
-L LED D2
+L LED D1
 U 1 1 4FD32F16
 P 3450 9850
-F 0 "D2" H 3450 9950 50  0000 C CNN
+F 0 "D1" H 3450 9950 50  0000 C CNN
 F 1 "RSSI" H 3450 9750 50  0000 C CNN
 	1    3450 9850
@@
 $EndComp
 $Comp
-L LED D5
+L LED D4
 U 1 1 4FD74922
 P 8850 9800
-F 0 "D5" H 8850 9900 50  0000 C CNN
+F 0 "D4" H 8850 9900 50  0000 C CNN
 F 1 "IR_LED" H 8850 9700 50  0000 C CNN
 	1    8850 9800
@@
 $EndComp
 $Comp
-L LED D6
+L LED D5
 U 1 1 4FD766BB
 P 9750 9800
-F 0 "D6" H 9750 9900 50  0000 C CNN
+F 0 "D5" H 9750 9900 50  0000 C CNN
 F 1 "IR_LED" H 9750 9700 50  0000 C CNN
 	1    9750 9800
@@
 $EndComp
 $Comp
-L LED D7
+L LED D6
 U 1 1 4FD766E4
 P 10650 9800
-F 0 "D7" H 10650 9900 50  0000 C CNN
+F 0 "D6" H 10650 9900 50  0000 C CNN
 F 1 "IR_LED" H 10650 9700 50  0000 C CNN
 	1    10650 9800
@@
 $EndComp
 $Comp
-L LED D8
+L LED D7
 U 1 1 4FD7670D
 P 11550 9800
-F 0 "D8" H 11550 9900 50  0000 C CNN
+F 0 "D7" H 11550 9900 50  0000 C CNN
 F 1 "IR_LED" H 11550 9700 50  0000 C CNN
 	1    11550 9800
@@
 ENC_RB
 $Comp
-L LED D9
+L LED D8
 U 1 1 4FE0E9A1
 P 15700 5500
-F 0 "D9" H 15700 5600 50  0000 C CNN
+F 0 "D8" H 15700 5600 50  0000 C CNN
 F 1 "IR_LD271" H 15700 5400 50  0000 C CNN
 	1    15700 5500
@@
 $EndComp
 $Comp
-L LED D10
+L LED D9
 U 1 1 4FE0E9C5
 P 15700 5900
-F 0 "D10" H 15700 6000 50  0000 C CNN
+F 0 "D9" H 15700 6000 50  0000 C CNN
 F 1 "IR_LD271" H 15700 5800 50  0000 C CNN
 	1    15700 5900
@@
 $EndComp
 $Comp
-L LED D11
+L LED D10
 U 1 1 4FE0E9CB
 P 15700 6300
-F 0 "D11" H 15700 6400 50  0000 C CNN
+F 0 "D10" H 15700 6400 50  0000 C CNN
 F 1 "IR_LD271" H 15700 6200 50  0000 C CNN
 	1    15700 6300
@@
 5V_IR
 $Comp
-L ULN2003A U5
+L ULN2003A U6
 U 1 1 4FE0F20E
 P 13950 4800
-F 0 "U5" H 13950 4900 70  0000 C CNN
+F 0 "U6" H 13950 4900 70  0000 C CNN
 F 1 "ULN2003A" H 13950 5350 70  0000 C CNN
 	1    13950 4800
@@
 $EndComp
 $Comp
-L DIODE D1
+L DIODE InvPolDiode1
 U 1 1 4FE4BC6C
 P 3100 2250
-F 0 "D1" H 3100 2350 40  0000 C CNN
-F 1 "InvPolarity" H 3100 2150 40  0000 C CNN
+F 0 "InvPolDiode1" H 3100 2350 40  0000 C CNN
+F 1 "200mA min" H 3100 2150 40  0000 C CNN
 	1    3100 2250
 	0    -1   -1   0
@@
 $EndComp
 $Comp
-L LED D4
+L LED D3
 U 1 1 4FE4BCA1
 P 6750 2300
-F 0 "D4" H 6750 2400 50  0000 C CNN
+F 0 "D3" H 6750 2400 50  0000 C CNN
 F 1 "ON" H 6750 2200 50  0000 C CNN
 	1    6750 2300
@@
 	1    0    0    -1
 $EndComp
-Text Notes 2450 2100 0    58   Italic 12
-Test the IPP!
 Text Label 8450 6300 2    58   ~ 0
 5V_IRScanner
@@
 	2850 4700 3150 4700
 $Comp
-L INDUCTOR 10uH1
+L INDUCTOR U1
 U 1 1 4FE85F66
 P 2550 4700
-F 0 "10uH1" V 2500 4700 40  0000 C CNN
+F 0 "U1" V 2500 4700 40  0000 C CNN
 F 1 "INDUCTOR" V 2650 4700 40  0000 C CNN
 	1    2550 4700
